Commit message: dagger_bringup: fused odom + Theta* + scan band fix -> straight path-following works
Odometry (odom_source:=fused, now the default):
- New robot_localization EKF (params/ekf_fused.yaml) on EK3 body VELOCITY +
  raw gyro yaw rate only -- no GPS position/yaw in odom. The GPS-anchored EK3
  pose (fcu mode) walked 1-3 m/min at rest and slid 1.7 m sideways during a
  20 s drive, so Nav2 steered the rover into a left arc chasing it.
- fcu_odom_relay: twist_variance (mavros sends all-zero covariance) and
  zero_velocity_deadband 0.02 m/s (EK3 5 mm/s rest bias -> 0.31 m/min creep;
  now 0.000 m over 30 s).

Planning / control:
- Planner SmacPlanner2D -> ThetaStarPlanner: the 8-connected grid turned a
  39.4 deg straight goal into 45 deg diagonals (0.40 m bulge left).
- RPP lookahead 0.6 -> 2.0 m (1.5-3.0), v 0.4, approach 1.0 m / 0.15 m/s,
  rotate 0.45, xy_goal_tolerance 0.5. 6 m straight: CTE 0.042 m RMS,
  1 cmd reversal, goal err 0.12 m (was 4 reversals, 0.36 m).

Perception / TF:
- dagger_description lidar_joint z 1.1 -> 0.92: LiDAR measured 1.12 m above
  ground (base_joint 0.2 was double-counted) -> flat ground read +0.19 m and
  the lowest-beam ground ring became a lethal wall in the costmap.
- pointcloud_to_laserscan band 0.15-0.90 -> 0.35-0.75 m: ground stays out,
  and mast self-returns (now z 0.81+) no longer abort Spin "Collision Ahead".
  Stopgap until proper ground segmentation.

Validated on vehicle: 6 m straight out + Nav2 /spin 180 (178.5 deg, 0 sign
flips, SUCCEEDED) + return to start.

tools/: preflight.py (stream rates + health gate), pf_record.sh,
pf_analyze.py, send_goal.py, pf_tune.sh, estop.sh / estop_clear.sh.

File: src/dagger_description/urdf/robot.urdf.xacro (robot description, xacro)
@@ -309,6 +309,9 @@
     name="lidar_joint"
     type="fixed">
-    <origin
-      xyz="0.2925 0 1.1"
+    <!-- z 1.1 -> 0.92 (2026-09-14): LiDAR measured 1.12 m above ground; base_joint
+         already puts base_link 0.2 m up, so 1.1 double-counted it (1.30 m total)
+         and flat ground read +0.19 m -> ground ring became costmap obstacles. -->
+    <origin
+      xyz="0.2925 0 0.92"
       rpy="0 0 1.5708" />
     <parent

Commit message: dagger_description: D435 camera link, so a detection bearing has a frame
User measured the lens centre at 0.99 m above ground, aimed dead ahead with no
pitch, mounted directly below the LiDAR. base_joint already lifts base_link
0.2 m, so the joint is z 0.79; the LiDAR's 1.12 m is 0.92 by the same
arithmetic, putting the camera 0.13 m below it. x is taken from the LiDAR since
the camera hangs under it, y is 0.

Of the three, y is the one that matters: a lateral error becomes a bearing error
directly (0.05 m off centre is 1 degree at 3 m), while an error along x is
almost purely radial and barely moves the bearing.

The child link has to be d435_link -- the driver derives its frame prefix from
camera_name and publishes d435_link -> d435_color_optical_frame itself, so this
joint is what attaches that subtree to the robot. Without it there is no
base_footprint -> camera transform at all and a bearing cannot be turned into a
LiDAR direction.

Verified live against the running driver:
  base_footprint -> d435_link                (0.2925, 0.0000, 0.9900) yaw 0.0
  base_footprint -> d435_color_optical_frame (0.2925, 0.0147, 0.9902) yaw -89.8
  base_footprint -> lidar_link               (0.2925, 0.0000, 1.1200)
The 14.7 mm on y is the factory offset from the depth imager to the colour one,
which is exactly why the selector transforms through TF instead of assuming the
lens is on the centreline.

robot_state_publisher takes a live robot_description update, but a T1 restart is
the simple way to pick this up.

File: src/dagger_description/urdf/robot.urdf.xacro (robot description, xacro)
@@ -319,4 +319,46 @@
     <child
       link="lidar_link" />
+    <axis
+      xyz="0 0 0" />
+  </joint>
+  <!-- Intel RealSense D435, follow-me detector camera (added 2026-09-25).
+       Measured by the user: lens centre 0.99 m above ground, aimed dead ahead
+       with no pitch, mounted directly below the LiDAR. base_joint already lifts
+       base_link 0.2 m, so z here is 0.99 - 0.2 = 0.79 (the LiDAR's 1.12 m is
+       0.92 by the same arithmetic; the camera sits 0.13 m below it).
+       x is taken from the LiDAR's 0.2925 since the camera is mounted under it,
+       and y is 0. Of the three, y is the one that matters: a lateral error
+       becomes a bearing error directly (0.05 m off centre = 1 deg at 3 m),
+       while an error along x is almost purely radial and barely moves the
+       bearing at all.
+       The child link name must stay d435_link: the driver derives its own frame
+       prefix from the camera_name parameter (parameters.cpp:83) and publishes
+       d435_link -> d435_color_optical_frame itself, so this joint is what
+       connects that subtree to the robot. Without it a detection bearing cannot
+       be transformed into the LiDAR's frame at all.
+       The D435's own camera_link sits at the depth (left) imager rather than the
+       physical lens centre, roughly 1-2 cm away. At 3 m that is under half a
+       degree, well inside what the bearing needs. -->
+  <link name="d435_link">
+    <visual>
+      <origin xyz="0 0 0" rpy="0 0 0" />
+      <geometry>
+        <box size="0.025 0.090 0.025" />
+      </geometry>
+      <material name="">
+        <color rgba="0.1 0.1 0.1 1" />
+      </material>
+    </visual>
+  </link>
+  <joint
+    name="d435_joint"
+    type="fixed">
+    <origin
+      xyz="0.2925 0 0.79"
+      rpy="0 0 0" />
+    <parent
+      link="base_link" />
+    <child
+      link="d435_link" />
     <axis
       xyz="0 0 0" />
